File: pcb/ovc.sch (KiCad schematic (older format))
At the start: 188 parts

Commit message: added connections to ucontroller
Parts:
- removed Q? (x3): MMBT3906LT1G, digikey-footprints:SOT-23-3, symbol dk_Transistors-Bipolar-BJT-Single:MMBT3906LT1G
- removed R?: R, VC:VC-RES-0603-1608metric, symbol Device:R
- added C?: C, symbol Device:C
- added C?: 470nF, symbol Device:C
- added J?: Conn_02x03_Counter_Clockwise, symbol Connector_Generic:Conn_02x03_Counter_Clockwise
- added U?: SN74LVC3G17, VC:TexasInstruments_DCU8_R-PDSO-G8_0.5mm, symbol vc_misc:SN74LVC3G17
Connections:
- net labels added: PGEC1, PGED1, SQICLK, SQICS1, SQID0, SQID1, SQID2, SQID3
- wire segments 921 -> 938
Other:
- note added: "agregar pull ups pull downs, headers, botones, leds y puertos para display: 16x2 y 4Dsystems, agregar memoria sqi, header de programación"
- moved on the sheet: C?, R?, U?

Commit message: added memory pull ups connectors and memory ic
Parts:
- removed R? (x3): 5k, VC:VC-RES-0603-1608metric, symbol Device:R
- added C?: 100nF, symbol Device:C
- added C?: 10uF, symbol Device:C
- added D? (x4): LTST-C191KRKT, digikey-footprints:LED_0603, symbol dk_LED-Indication-Discrete:LTST-C191KRKT
- added J?: Conn_02x10_Odd_Even, symbol Connector_Generic:Conn_02x10_Odd_Even
- added R? (x29): 10k, VC:VC-RES-0603-1608metric, symbol Device:R
- added R? (x8): 330, VC:VC-RES-0603-1608metric, symbol Device:R
- added S? (x4): B3U-1000P, digikey-footprints:Switch_Tactile_SMD_B3U-1000P, symbol dk_Tactile-Switches:B3U-1000P
- added U?: SST26VF032BA-V104I_SM, VC:Microchip-SOIJ-8-1.27mm, symbol vc_misc:SST26VF032BA-V104I_SM
- R? (x2): value R -> 330
Connections:
- net +3.3VA: now also R?.1, R?.1, R?.1, R?.1, R?.1, R?.1, R?.1, R?.1, R?.1, R?.1
- net +3V3: now also C?.1, C?.1, R?.1, R?.1, R?.1, R?.1, R?.1, R?.1, R?.1, R?.1, U?.8 (VDD)
- net ADC-~RST~: now also R?.1
- net CJ-ALERT: now also R?.2, R?.2
- net CJ-SCL: now also R?.2, R?.2
- net CJ-SDA: now also R?.2, R?.2
- net GND: now also C?.2, C?.2, D?.1, D?.1, D?.1, D?.1, R?.2, R?.2, R?.2, R?.2, R?.2, R?.2, R?.2, R?.2, R?.2, R?.2, R?.2, S?.1, S?.1, S?.1, S?.1, U?.4 (VSS)
- net M1-EN: now also R?.1
- net M2-EN: now also R?.1
- net M3-EN: now also R?.1
- net M4-EN: now also R?.1
- net M5-EN: now also R?.1
- net SD_~CS~: now also R?.1
- net SQICLK: now also U?.6 (SCK)
- net SQICS1: now also R?.1, U?.1 (CE#)
- net SQID0: now also U?.5 (SIO0/SI)
- net SQID1: now also U?.2 (SIO1/SO)
- net SQID2: now also U?.3 (SIO2/WP#)
- net SQID3: now also U?.7 (SIO3/HOLD)
- net W-RX: now also R?.1
- net W-TX: now also R?.1
- net W_EN: now also R?.1
- net LED1: now reaches U?.26 (RB6/AN46/RPB6/PGEC2)
- net LED1: now also R?.1
- net LED2: now reaches U?.27 (RB7/AN47/RPB7/PGED2)
- net LED2: now also R?.1
- net LED3: now reaches U?.28 (RA9/AN27/VREF-/CVREF-/AERXD2)
- net LED3: now also R?.1
- net LED4: now reaches U?.29 (RA10/AN28/VREF+/CVREF+/AERXD3)
- net LED4: now also R?.1
- net SW1: now reaches U?.35 (RB11/AN6/AETXERR/ERXERR)
- net SW1: now also R?.1
- net SW2: now reaches U?.47 (RD14/AN32/RPD14/AETXD0)
- net SW2: now also R?.1
- net SW3: now reaches U?.48 (RD15/AN33/SCK6/RPD15/AETXD1)
- net SW3: now also R?.1
- net SW4: now reaches U?.50 (RC15/OSC2/CLKO)
- net SW4: now also R?.1
- net SDA3: now reaches U?.57 (RF2/SDA3/RPF2/EBIRDY3)
- net SDA3: now also R?.2, R?.2
- net SCL3: now reaches U?.58 (RF8/SCL3/RPF8/EBIRDY2)
- net SCL3: now also R?.2, R?.2
- net SCL2: now reaches U?.59 (RA2/SCL2/EBICS0)
- net SCL2: now also R?.2, R?.2
- net SDA2: now reaches U?.60 (RA3/SDA2/EBIRDY1)
- net SDA2: now also R?.2, R?.2
- new net: R?.2, R?.2, S?.2 (x4)
- new net: D?.2, R?.2 (x4)
Other:
- note added: "Place close to connector for junction temperature compensation"
- note added: "Place close to miccrocontroller, \navoid vias and try to match wire lenght."
- note added: "agregar:\n- headers\n- puertos para display: \n *O128O064DGPP3N0000\n *4Dsystems\n\n"
- note removed: "agregar pull ups pull downs, headers, botones, leds y puertos para display: 16x2 y 4Dsystems, agregar memoria sqi, header de programación"
- moved on the sheet: C?, D?, J?, JP?, R?, U?
