File: pcb/ovc.kicad_pcb (KiCad board)
At the start: 2 copper layers, 90 x 80 mm, 270 parts, among them J1 Conn_01x12, J10 Conn_01x04, J11 Conn_01x04, J12 Conn_02x10_Odd_Even, J13 Conn_02x11_Odd_Even, J14 Conn_01x04, J15 Conn_01x04, J16 Conn_01x31, J17 12401610E4_2A, J18 Conn_01x13, J19 Conn_01x14, J2 Micro_SD_Card_Det_Hirose_DM3AT, J20 Conn_01x06, J21 Conn_01x08, J22 Conn_01x08, J23 Conn_01x10, J3 Conn_02x04_Counter_Clockwise, J4 Conn_01x04, J5 Conn_01x04, J6 Conn_01x02, J7 Conn_01x04, J8 Conn_01x04, J9 Conn_01x02, Q1 MMBT3906, Q10 MMBT3906, Q11 MMBT3906, Q12 MMBT3906, Q2 MMBT3906, Q3 IRLML6401TRPBF, Q4 IRLML6401TRPBF, Q5 IRLML6401TRPBF, Q6 DMT6016LSS, Q7 DMT6016LSS, Q8 MMBT3906, Q9 MMBT3906, U1 SST26VF032BA-V104I_SM, U10 MAX31856, U11 L7805CV, U12 AP2112K-3.3, U13 SN74HC595N, U14 ESP32-WROOM-32D, U15 SN74HC595N, U2 SN74LVC3G17, U3 ADS1248, U4 PIC32MZ1024EFK100-PF, U5 ASDK2-32.768KHZ-LR-T3, U6 ASEM1-12.000MHZ-LC-T, U7 SN74LVC3G17, U8 TMP112AIDRLT, U9 AP2112K-3.3

Commit message: finished schematic, layed out components in pcb and advanced in routing
Parts:
- removed J19: Conn_01x14, Connector_PinHeader_2.54mm:PinHeader_1x14_P2.54mm_Vertical_SMD_Pin1Left
- removed J21, J22: Conn_01x08, Connector_PinHeader_2.54mm:PinHeader_1x08_P2.54mm_Vertical
- added C87: 10uF, VC:murata-CAP-GRM-0805-2012metric-reflow, F.Cu at (143.2, 99.8)
- added D28: MBR2H200SFT3G, VC:onsemi-sod123fl, F.Cu at (133.0, 115.2)
- added D29: LTST-C191KRKT, digikey-footprints:LED_0603, B.Cu at (128.9, 125.0)
- added DS1: LTC-4627JF, VC:liteon-C4627JF, B.Cu at (165.8, 115.7)
- added Q13: FDV301N, digikey-footprints:SOT-23-3, F.Cu at (132.0, 112.2)
- added R96: 10k, VC:VC-RES-0603-1608metric, F.Cu at (134.8, 112.2)
- added R97: 330, VC:VC-RES-0603-1608metric, B.Cu at (130.3, 125.0)
- added RLY3: G6DN-1A-L_DC5, VC:Omron G6DN-1A, B.Cu at (134.2, 117.6)
- C21, C41, C42, C53, C54, C60, C61, C63, C64, C66, C67, C71, C72, C74, C75, D23, D24, D25, D26, D27, J10, J11, J12, J20, J5, J6, J7, J8, JP1, Q10, Q11, Q12, Q8, Q9, R10, R19, R20, R21, R22, R23, R24, R25, R26, R62, R63, R64, R66, R67, R68, R74, R75, R76, R77, R78, R79, R80, R81, R82, R83, R84, R85, R86, R87, R88, R9, R91, R92, R93, R94, R95, RLY1, RLY2, S1, S2, S3, S4, U11: moved to B.Cu
- C50: value 100nF -> 10uF; footprint VC:murata-CAP-GCM-0603-1608metric-reflow -> VC:murata-CAP-GRM-0805-2012metric-reflow
- C51: value 47uF -> 10uF; footprint Capacitor_SMD:C_Elec_6.3x5.8 -> VC:murata-CAP-GRM-0805-2012metric-reflow
- J1: value Conn_01x12 -> Conn_01x13; footprint VC:phoenix_contact-therminal_block-12pos_PTSA1.5_12-3.5-F-1985069 -> VC:phoenix_contact-therminal_block-13pos_PTSA1.5_13-3.5-F-1985072
- J13: footprint Connector_PinHeader_2.54mm:PinHeader_2x11_P2.54mm_Vertical_SMD -> Connector_PinHeader_2.54mm:PinHeader_2x12_P2.54mm_Vertical_SMD; moved to B.Cu
- J14: value Conn_01x04 -> Conn_02x18_Odd_Even; footprint Connector_PinHeader_2.54mm:PinHeader_1x04_P2.54mm_Vertical -> Connector_PinHeader_2.54mm:PinHeader_2x18_P2.54mm_Vertical_SMD; moved to B.Cu
- J15: value Conn_01x04 -> Conn_01x02; footprint Connector_PinHeader_2.54mm:PinHeader_1x04_P2.54mm_Vertical -> VC:phoenix_contact-therminal_block-2pos_PTSA1.5-2-3.5-F-1984963; moved to B.Cu
- J18: value Conn_01x13 -> Conn_02x03_Odd_Even; footprint Connector_PinHeader_2.54mm:PinHeader_1x13_P2.54mm_Vertical_SMD_Pin1Left -> Connector_PinHeader_2.54mm:PinHeader_2x03_P2.54mm_Vertical; moved to B.Cu
- J4: footprint Connector_Phoenix_MSTB:PhoenixContact_MSTBA_2,5_4-G_1x04_P5.00mm_Horizontal -> VC:phoenix_contact-therminal_block-4pos_PTSA1.5-4-3.5-F-1984989; moved to B.Cu
- J9: value Conn_01x02 -> Conn_01x04; footprint Connector_Phoenix_MSTB:PhoenixContact_MSTBA_2,5_2-G_1x02_P5.00mm_Horizontal -> VC:phoenix_contact-therminal_block-4pos_PTSA1.5-4-3.5-F-1984989; moved to B.Cu
- U13, U15: footprint digikey-footprints:DIP-16_W7.62mm -> digikey-footprints:SOIC-16_W3.90mm
- moved R30 237.5 mm to (131.5, 102.3)
- moved C55 235.8 mm to (137.6, 99.8), turned to 90 degrees
- moved C56 234.8 mm to (136.0, 100.0), turned to 90 degrees
- moved C6 229.9 mm to (146.4, 81.6)
- moved R13 225.6 mm to (135.6, 123.1), turned to 270 degrees
- moved J15 222.7 mm to (119.7, 125.0), turned to 90 degrees
- moved C51 222.0 mm to (136.4, 116.6), turned to 90 degrees
- moved C66 219.9 mm to (144.8, 76.2), turned to 270 degrees
- moved C32 213.3 mm to (134.5, 104.7)
- moved R63 211.9 mm to (156.0, 115.9), turned to 180 degrees
- moved R90 211.6 mm to (164.1, 109.2)
- moved R64 208.3 mm to (147.2, 113.0), turned to 180 degrees
- moved R75 203.1 mm to (164.6, 115.7), turned to 180 degrees
- moved R1 202.4 mm to (165.8, 71.1)
- moved R73 202.4 mm to (169.8, 61.6)
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Connections:
- net /BRD1_P renamed /BRDN2_P
- net /BRD2_P renamed /BRDN1_P
- net /TH2-I1 renamed /TH2-N
- net /TH2-I2 renamed /TH2-P
- net Net-(D11-PadK) renamed /THPF_N
- net Net-(D13-PadA) renamed /THPF_P
- C33 pad 1: /TH1-I1 -> /TH1_N
- C34 pad 1: /THERM_P -> /THERM_N
- C35 pad 1: /TH1-I1 -> /TH1_N
- C35 pad 2: /TH1-I2 -> /TH1_P
- C36 pad 1: /THERM_P -> /THERM_N
- C36 pad 2: /THERM_N -> /THERM_P
- C37 pad 2: /TH1-I2 -> /TH1_P
- C38 pad 2: /THERM_N -> /THERM_P
- C51 pad 1: VDD -> +5V
- C6 pad 1: +3V3 -> +5V
- C76 pad 2: /BRDN1_N -> /BRDN2_N
- C81 pad 2: /BRDN2_N -> /BRDN1_N
- D10 pad 1: /TH1-I1 -> /TH1_N
- D15 pad 1: /TH1-I2 -> /TH1_P
- D17 pad 1: /D+ -> /D-
- D17 pad 3: /D- -> /D+
- D17 pad 4: /DD- -> /DD+
- D17 pad 6: /DD+ -> /DD-
- J1 pad 10: Net-(C23-Pad1) -> Net-(C25-Pad1)
- J1 pad 11: Net-(C15-Pad1) -> Net-(C23-Pad1)
- J1 pad 12: Net-(C8-Pad1) -> Net-(C15-Pad1)
- J1 pad 3: /TH1-I2 -> /TH1_P
- J1 pad 4: /TH1-I1 -> /TH1_N
- J1 pad 5: /CIN-2 -> GND
- J1 pad 6: +24V -> /CIN-1
- J1 pad 7: /CIN-1 -> +24V
- J1 pad 8: +24V -> /CIN-2
- J1 pad 9: Net-(C25-Pad1) -> +24V
- J12 pad 15: /RE0 -> +5V
- J14 pad 3: GND -> +3V3
- J14 pad 4: GND -> +3V3
- J15 pad 1: +3V3 -> Net-(J15-Pad1)
- J15 pad 2: +3V3 -> Net-(J15-Pad2)
- J18 pad 1: /W_EN -> +3V3
- J18 pad 2: /W-SVP -> GND
- J18 pad 3: /W-SVN -> +3.3VA
- J18 pad 4: /W-IO34 -> GND
- J18 pad 5: /W-IO35 -> +5V
- J18 pad 6: /W-IO32 -> GND
- J9 pad 2: GND -> +12V
- Q10 pad 3: /CA-1 -> /CA-4
- Q11 pad 3: /CA-3 -> /CA-2
- Q12 pad 3: /CA-2 -> /CA-3
- Q8 pad 3: /CA-4 -> /CA-1
- R25 pad 2: /SCL3 -> /MCURX-SCL3
- R26 pad 2: /SCL3 -> /MCURX-SCL3
- R27 pad 2: /TH1-I1 -> /TH1_N
- R28 pad 1: /THERM_P -> /THERM_N
- R31 pad 2: /TH1-I2 -> /TH1_N
- R32 pad 2: /TH1-I2 -> /TH1_P
- R33 pad 1: /THERM_N -> /THERM_P
- R34 pad 1: /TH1-I2 -> /TH1_N
- R51 pad 2: Net-(Q6-Pad1) -> Net-(Q7-Pad1)
- R52 pad 1: Net-(Q6-Pad1) -> Net-(Q7-Pad1)
- R52 pad 2: Net-(D21-Pad2) -> Net-(D21-Pad1)
- R53 pad 1: /BRDN1_N -> /BRDN2_N
- R53 pad 2: Net-(D21-Pad2) -> Net-(D21-Pad1)
- R57 pad 2: Net-(Q7-Pad1) -> Net-(Q6-Pad1)
- R61 pad 1: Net-(Q7-Pad1) -> Net-(Q6-Pad1)
- R61 pad 2: Net-(D21-Pad1) -> Net-(D21-Pad2)
- R65 pad 1: /BRDN2_N -> /BRDN1_N
- R65 pad 2: Net-(D21-Pad1) -> Net-(D21-Pad2)
- R93 pad 1: /DP -> /D
- R95 pad 1: /D -> /DP
- U2 pad 8: +3V3 -> +5V
- U3 pad 14: /BRDN1_N -> /BRDN2_N
- U3 pad 16: /BRDN2_N -> /BRDN1_N
- U3 pad 17: /THERM_P -> /THERM_N
- U3 pad 18: /THERM_N -> /THERM_P
- U4 pad 20: /CLKI -> (no net)
Routing:
- net GND: track 0.00 -> 105.1 mm, vias 0 -> 101
- net /AN-MISO: track 0.00 -> 75.2 mm, vias 0 -> 2
- net /AN-MOSI: track 0.00 -> 74.9 mm, vias 0 -> 2
- net /SDA3: track 0.00 -> 61.7 mm, vias 0 -> 1
- net /MCLR: track 0.00 -> 58.4 mm, vias 0 -> 3
- net /MCURX-SCL3: track 0.00 -> 56.4 mm, vias 0 -> 1
- net /CJ-ALERT: track 0.00 -> 55.4 mm, vias 0 -> 2
- net /CJ-SDA: track 0.00 -> 55.2 mm, vias 0 -> 2
- net /DD-: track 0.00 -> 52.8 mm
- net /DD+: track 0.00 -> 52.2 mm
- net /CJ-SCL: track 0.00 -> 51.6 mm, vias 0 -> 2
- net /ADC-CS: track 0.00 -> 50.9 mm, vias 0 -> 2
- net /RB15: track 0.00 -> 47.7 mm, vias 0 -> 1
- net /AN-SCLK: track 0.00 -> 47.6 mm, vias 0 -> 1
- net /ADC-~RST~: track 0.00 -> 44.9 mm, vias 0 -> 2
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- added copper zone on F.Cu, net GND
- added copper zone on In1.Cu, net GND
Other:
- board size 90 x 80 mm -> 120 x 80 mm
- copper layers 2 -> 4
- net class Default: clearance 0.2 -> 0.15; trace_width 0.25 -> 0.15; via_dia 0.8 -> 0.6; via_drill 0.4 -> 0.35
- rule pad_to_mask_clearance: 0.051 -> 0.03
- rule solder_mask_min_width: 0.25 -> 0.07
- rule trace_clearance: 0.2 -> 0.15
- rule trace_min: 0.2 -> 0.15
- rule via_min_drill: 0.3 -> 0.35
- rule via_min_size: 0.4 -> 0.6

Commit message: gerber generated and fabricated
Parts:
- removed J4: Conn_01x04, VC:phoenix_contact-therminal_block-4pos_PTSA1.5-4-3.5-F-1984989
- added C88: 10uF, VC:murata-CAP-GRM-0805-2012metric-reflow, F.Cu at (146.9, 54.6)
- added C89: 10uF, VC:murata-CAP-GRM-0805-2012metric-reflow, F.Cu at (228.3, 93.1)
- added REF**: 2.5mm-screw-Hole, VC:2.5mm-screw-Hole, B.Cu at (165.0, 126.1)
- C84, R59, R60, R72: moved to B.Cu
- J1: value Conn_01x13 -> Conn_01x16; footprint VC:phoenix_contact-therminal_block-13pos_PTSA1.5_13-3.5-F-1985072 -> VC:phoenix_contact-therminal_block-16pos_PTSA1.5_16-3.5-F-1985108
- J20: footprint Connector_PinHeader_1.27mm:PinHeader_1x06_P1.27mm_Vertical_SMD_Pin1Left -> Connector_PinHeader_1.27mm:PinHeader_1x06_P1.27mm_Vertical_SMD_Pin1Right
- moved R42 54.5 mm to (190.2, 53.0), turned to 270 degrees
- moved R40 50.9 mm to (222.0, 53.0), turned to 270 degrees
- moved R41 45.8 mm to (206.2, 53.0), turned to 270 degrees
- moved R39 33.5 mm to (222.0, 73.2), turned to 270 degrees
- moved R59 31.9 mm to (183.4, 109.6)
- moved R60 31.6 mm to (183.4, 108.4)
- moved R58 20.2 mm to (201.2, 118.2), turned to 90 degrees
- moved C85 18.5 mm to (233.5, 122.7), turned to 0 degrees
- moved R38 18.4 mm to (222.0, 94.2), turned to 270 degrees
- moved R76 17.6 mm to (163.2, 106.7), turned to 0 degrees
- moved R74 17.6 mm to (160.6, 106.7)
- moved R87 17.6 mm to (180.8, 106.6), turned to 0 degrees
- moved R86 17.6 mm to (178.2, 106.6)
- moved R69 11.8 mm to (174.8, 122.3), turned to 0 degrees
- moved J6 8.84 mm to (197.3, 73.3), turned to 90 degrees
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Connections:
- A4 pad 12: /M5-CS -> /M4-CS
- A4 pad 15: /M5-STP -> /M4-STP
- A4 pad 16: /M5-DIR -> /M4-DIR
- A4 pad 9: /M5-EN -> /M4-EN
- A5 pad 12: /M4-CS -> /M5-CS
- A5 pad 15: /M4-STP -> /M5-STP
- A5 pad 16: /M4-DIR -> /M5-DIR
- A5 pad 9: /M4-EN -> /M5-EN
- D12 pad 1: Net-(D12-Pad1) -> /SSRD-1
- D14 pad 1: Net-(D14-Pad1) -> /SSRD-2
- J1 pad 1: /TH2-P -> /SSRD-1
- J1 pad 10: Net-(C25-Pad1) -> +24V
- J1 pad 11: Net-(C23-Pad1) -> /CIN-2
- J1 pad 12: Net-(C15-Pad1) -> +24V
- J1 pad 13: Net-(C8-Pad1) -> Net-(C25-Pad1)
- J1 pad 2: /TH2-N -> /SSRD-2
- J1 pad 3: /TH1_P -> GND
- J1 pad 4: /TH1_N -> /TH2-P
- J1 pad 5: GND -> /TH2-N
- J1 pad 6: /CIN-1 -> /TH1_P
- J1 pad 7: +24V -> /TH1_N
- J1 pad 8: /CIN-2 -> GND
- J1 pad 9: +24V -> /CIN-1
- J14 pad 10: /W-IO23 -> GND
- J14 pad 11: /W_EN -> /W-IO22
- J14 pad 12: /W-IO22 -> /W_EN
- J14 pad 13: /W-SVP -> /W-IO1
- J14 pad 14: /W-IO1 -> /W-SVP
- J14 pad 15: /W-SVN -> /W-IO3
- J14 pad 16: /W-IO3 -> /W-SVN
- J14 pad 17: /W-IO34 -> /W-IO21
- J14 pad 18: /W-IO21 -> /W-IO34
- J14 pad 19: /W-IO35 -> /W-IO19
- J14 pad 20: /W-IO19 -> /W-IO35
- J14 pad 21: /W-IO32 -> /W-IO18
- J14 pad 22: /W-IO18 -> /W-IO32
- J14 pad 23: /W-IO33 -> /W-IO5
- J14 pad 24: /W-IO5 -> /W-IO33
- J14 pad 25: /W-IO25 -> /W-TX
- J14 pad 26: /W-TX -> /W-IO25
- J14 pad 27: /W-IO26 -> /W-RX
- J14 pad 28: /W-RX -> /W-IO26
- J14 pad 29: /W-IO27 -> /W-IO4
- J14 pad 30: /W-IO4 -> /W-IO27
- J14 pad 31: /W-RTS -> /W-BOOT
- J14 pad 32: /W-BOOT -> /W-RTS
- J14 pad 33: /W-TX0 -> /W-IO2
- J14 pad 34: /W-IO2 -> /W-TX0
- J14 pad 35: /W-RX0 -> /W-CTS
- J14 pad 36: /W-CTS -> /W-RX0
- J14 pad 9: GND -> /W-IO23
- J16 pad 13: Net-(J13-Pad22) -> Net-(J13-Pad12)
- J16 pad 14: Net-(J13-Pad20) -> Net-(J13-Pad10)
- J16 pad 15: Net-(J13-Pad18) -> Net-(J13-Pad8)
- J16 pad 18: Net-(J13-Pad12) -> Net-(J13-Pad18)
- J16 pad 19: Net-(J13-Pad10) -> Net-(J13-Pad20)
- J16 pad 20: Net-(J13-Pad8) -> Net-(J13-Pad22)
- J18 pad 3: +3.3VA -> +3V3
- R29 pad 1: Net-(D12-Pad1) -> /SSRD-1
- R30 pad 1: Net-(D14-Pad1) -> /SSRD-2
- R62 pad 1: +3.3VA -> +3V3
- R74 pad 1: +3.3VA -> +3V3
- R80 pad 1: +3.3VA -> +3V3
- R86 pad 1: +3.3VA -> +3V3
- U4 pad 100: /M5-STP -> /M5-EN
- U4 pad 64: /M1-EN -> /M1-DIR
- U4 pad 66: /M1-DIR -> /M1-CS
- U4 pad 68: /M1-CS -> /M1-EN
- U4 pad 71: /M2-EN -> /M2-DIR
- U4 pad 73: /M2-CS -> /M2-STP
- U4 pad 76: /M2-STP -> /M2-CS
- U4 pad 77: /M2-DIR -> /M2-EN
- U4 pad 94: /M5-EN -> /M5-DIR
- U4 pad 98: /M5-CS -> /M5-STP
- U4 pad 99: /M5-DIR -> /M5-CS
Routing:
- net +3V3: track 24.8 -> 351.1 mm, vias 3 -> 38
- net +5V: track 25.5 -> 195.4 mm, vias 3 -> 24
- net /M-MISO: track 0.00 -> 127.4 mm, vias 0 -> 3
- net /M-MOSI: track 0.00 -> 126.9 mm, vias 0 -> 4
- net /M-SCK: track 0.00 -> 122.5 mm, vias 0 -> 4
- net GND: track 105.1 -> 187.4 mm, vias 101 -> 216
- net /MCURX-SCL3: track 56.4 -> 133.0 mm, vias 1 -> 3
- net /4DRST-A4: track 34.6 -> 108.7 mm, vias 3 -> 5
- net /MCUTX-F3: track 36.2 -> 107.9 mm, vias 3 -> 5
- net /W_EN: track 0.00 -> 71.3 mm, vias 0 -> 3
- net /M3-EN: track 0.00 -> 69.3 mm, vias 0 -> 1
- net /W-BOOT: track 0.00 -> 67.9 mm, vias 0 -> 3
- net /M2-STP: track 0.00 -> 63.4 mm, vias 0 -> 1
- net /M3-CS: track 0.00 -> 63.3 mm, vias 0 -> 1
- net /M2-DIR: track 0.00 -> 63.1 mm, vias 0 -> 1
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- added copper zone on B.Cu, net +12V
- added copper zone on In2.Cu, net +12V
- added copper zone on F.Cu, net +3.3VA
- added copper zone on In2.Cu, net +3V3
- added copper zone on F.Cu, net +5V
- added copper zone on In2.Cu, net +5V
- added copper zone on B.Cu, net GND
- added copper zone on F.Cu, net Net-(Q3-Pad3)
- added copper zone on F.Cu, net VBUS
- added copper zone on In2.Cu, net VBUS
Other:
- outline, holes or cut-outs redrawn
- board text added: "+24"
- board text added: "+3V3"
- board text added: "+5V"
- board text added: "24VDC max"
- board text added: "5VO-1"
- board text added: "5VO-2"
- board text added: "CIN1"
- board text added: "CIN2"
- board text added: "GND"
- board text added: "PGEC"
- board text added: "PGED"
- board text added: "RA4"
- board text added: "RB15"
- board text added: "RF12"
- board text added: "RF3"
- board text added: "RS+"
- board text added: "RS-"
- board text added: "RTD+"
- board text added: "RTD-"
- board text added: "SCL2"
- board text added: "SCL3"
- board text added: "SDA2"
- board text added: "SDA3"
- board text added: "TC1+"
- board text added: "TC1-"
- board text added: "TC2+"
- board text added: "TC2-"
- board text added: "WB"
- board text added: "WCTS"
- board text added: "WEN"
- board text added: "WIO1"
- board text added: "WIO18"
- board text added: "WIO19"
- board text added: "WIO2"
- board text added: "WIO21"
- board text added: "WIO22"
- board text added: "WIO23"
- board text added: "WIO25"
- board text added: "WIO26"
- board text added: "WIO27"
- board text added: "WIO3"
- board text added: "WIO32"
- board text added: "WIO33"
- board text added: "WIO34"
- board text added: "WIO35"
- board text added: "WIO4"
- board text added: "WIO5"
- board text added: "WRTS"
- board text added: "WRX"
- board text added: "WRX0"
- board text added: "WSVN"
- board text added: "WSVP"
- board text added: "WTX"
- board text added: "WTX0"
